Commit message: have project3 now displaying map and linking odom to map

File: project3/src/my_robot/urdf/my_robot.xacro (robot description, xacro)
@@ -27,109 +27,84 @@
       </geometry>
     </visual>
+    <collision name="back_caster_collision">
+      <origin rpy=" 0 0 0" xyz="-0.15 0 -0.05"/>
+      <geometry>
+        <sphere radius="0.0499"/>
+      </geometry>
+    </collision>
+    <visual name="back_caster_visual">
+      <origin rpy=" 0 0 0" xyz="-0.15 0 -0.05"/>
+      <geometry>
+        <sphere radius="0.05"/>
+      </geometry>
+    </visual>
+    <collision name="front_caster_collision">
+      <origin rpy=" 0 0 0" xyz="0.15 0 -0.05"/>
+      <geometry>
+        <sphere radius="0.0499"/>
+      </geometry>
+    </collision>
+    <visual name="front_caster_visual">
+      <origin rpy=" 0 0 0" xyz="0.15 0 -0.05"/>
+      <geometry>
+        <sphere radius="0.05"/>
+      </geometry>
+    </visual>
   </link>
   <!--   wheels  -->
-  <xacro:property name="length_wheel" value="0.05" />
-  <xacro:property name="radius_wheel" value="0.08" />
-  <!-- <xacro:property name="camera_link" value="0.05" />  -->
-  <xacro:macro name="default_inertial" params="mass">
-               <inertial>
-                       <mass value="${mass}" />
-                       <inertia ixx="1.0" ixy="0.0" ixz="0.0"
-                                iyy="1.0" iyz="0.0"
-                                izz="1.0" />
-               </inertial>
-  </xacro:macro>
-  <link name="wheel_1">
-      <visual>
-          <geometry>
-              <cylinder length="${length_wheel}" radius="${radius_wheel}"/>
-          </geometry>
-      <!-- <origin rpy="0 1.5 0" xyz="0.1 0.1 0"/> -->
-      <origin rpy="0 0 0" xyz="0 0 0"/>
-        <material name="black">
-        <color rgba="0 0 0 1"/>
-      </material>
-    </visual>
-    <collision>
+  <link name="left_wheel">
+    <inertial>
+      <mass value="5"/>
+      <origin rpy=" 0 1.5707 1.5707" xyz="0 0 0"/>
+      <inertia ixx="0.1" ixy="0" ixz="0" iyy="0.1" iyz="0" izz="0.1"/>
+    </inertial>
+    <collision name="collision">
+      <origin rpy=" 0 1.5707 1.5707" xyz="0 0 0"/>
       <geometry>
-              <cylinder length="${length_wheel}" radius="${radius_wheel}"/>
+        <cylinder length="0.05" radius=".1"/>
       </geometry>
     </collision>
-    <xacro:default_inertial mass="1"/>
+    <visual name="chassis_visual">
+      <origin rpy=" 0 1.5707 1.5707" xyz="0 0 0"/>
+      <geometry>
+        <cylinder length="0.05" radius=".1"/>
+      </geometry>
+    </visual>
   </link>
-  <link name="wheel_2">
-      <visual>
-          <geometry>
-              <cylinder length="${length_wheel}" radius="${radius_wheel}"/>
-          </geometry>
-      <!-- <origin rpy="0 1.5 0" xyz="-0.1 0.1 0"/> -->
-      <origin rpy="0 0 0" xyz="0 0 0"/>
-        <material name="black"/>
-      </visual>
-    <collision>
+  <link name="right_wheel">
+    <inertial>
+      <mass value="5"/>
+      <origin rpy=" 0 1.5707 1.5707" xyz="0 0 0"/>
+      <inertia ixx="0.1" ixy="0" ixz="0" iyy="0.1" iyz="0" izz="0.1"/>
+    </inertial>
+    <collision name="collision">
+      <origin rpy=" 0 1.5707 1.5707" xyz="0 0 0"/>
       <geometry>
-              <cylinder length="${length_wheel}" radius="${radius_wheel}"/>
+        <cylinder length="0.05" radius=".1"/>
       </geometry>
     </collision>
-    <xacro:default_inertial mass="1"/>
+    <visual name="chassis_visual">
+      <origin rpy=" 0 1.5707 1.5707" xyz="0 0 0"/>
+      <geometry>
+        <cylinder length="0.05" radius=".1"/>
+      </geometry>
+    </visual>
   </link>
-  <link name="wheel_3">
-      <visual>
-          <geometry>
-              <cylinder length="${length_wheel}" radius="${radius_wheel}"/>
-          </geometry>
-      <!-- <origin rpy="0 1.5 0" xyz="0.1 -0.1 0"/> -->
-      <origin rpy="0 0 0" xyz="0 0 0"/>
-        <material name="black"/>
-      </visual>
-    <collision>
-      <geometry>
-              <cylinder length="${length_wheel}" radius="${radius_wheel}"/>
-      </geometry>
-    </collision>
-    <xacro:default_inertial mass="1"/>
-  </link>
-  <link name="wheel_4">
-      <visual>
-          <geometry>
-              <cylinder length="${length_wheel}" radius="${radius_wheel}"/>
-          </geometry>
-    <!--  <origin rpy="0 1.5 0" xyz="-0.1 -0.1 0"/> -->
-      <origin rpy="0 0 0" xyz="0 0 0" />
-        <material name="black"/>
-      </visual>
-    <collision>
-      <geometry>
-              <cylinder length="${length_wheel}" radius="${radius_wheel}"/>
-      </geometry>
-    </collision>
-    <xacro:default_inertial mass="1"/>
-  </link>
- <joint name="base_to_wheel1" type="continuous">
-   <parent link="chassis"/>
-   <child link="wheel_1"/>
-   <origin rpy="-1.5707 0 0" xyz="0.175 0.15 0"/>
-   <axis xyz="0 0 1" />
- </joint>
- <joint name="base_to_wheel2" type="continuous">
-   <axis xyz="0 0 1" />
-   <anchor xyz="0 0 0" />
-   <limit effort="100" velocity="100" />
-   <parent link="chassis"/>
-   <child link="wheel_2"/>
-   <origin rpy="-1.5707 0 0" xyz="-0.175 0.15 0"/>
-</joint>
- <joint name="base_to_wheel3" type="continuous">
-   <parent link="chassis"/>
-   <axis xyz="0 0 1" />
-   <child link="wheel_3"/>
-   <origin rpy="-1.5707 0 0" xyz="0.175 -0.15 0"/>
- </joint>
- <joint name="base_to_wheel4" type="continuous">
-   <parent link="chassis"/>
-   <axis xyz="0 0 1" />
-   <child link="wheel_4"/>
-   <origin rpy="-1.5707 0 0" xyz="-0.175 -0.15 0"/>
- </joint>
+  <joint name="left_wheel_hinge" type="continuous">
+    <origin rpy="0 0 0" xyz="0 0.15 0"/>
+    <child link="left_wheel"/>
+    <parent link="chassis"/>
+    <axis rpy="0 0 0" xyz="0 1 0"/>
+    <limit effort="10000" velocity="1000"/>
+    <dynamics damping="1.0" friction="1.0"/>
+  </joint>
+  <joint name="right_wheel_hinge" type="continuous">
+    <origin rpy="0 0 0" xyz="0 -0.15 0"/>
+    <child link="right_wheel"/>
+    <parent link="chassis"/>
+    <axis rpy="0 0 0" xyz="0 1 0"/>
+    <limit effort="10000" velocity="1000"/>
+    <dynamics damping="1.0" friction="1.0"/>
+  </joint>
   <link name="camera">
     <inertial>
